File: pnp/pcb/mobo/motor_control.sch (KiCad schematic (older format))
At the start: 37 parts, among them J1 X_MOTOR, J2 Y_MOTOR1, J3 Z_MOTOR, J37 P_MOTOR, J38 C_MOTOR, J4 R_MOTOR, J48 Y_MOTOR2

Commit message: Add 3v3 to pin 2 of motor driver for use with A4988 stepper driver
Connections:
- wire segments 168 -> 174
- no-connect marks 6 -> 0
