File: pnp/pcb/mobo/misc_input.sch (KiCad schematic (older format))
At the start: 9 parts, among them J18 R_LIMIT, J19 P_LIMIT, J20 C_LIMIT, J60 X_LIMIT, J61 Y_LIMIT, J62 Z_LIMIT, J65 ADC_AUX_1, J66 ADC_AUX_2, U6 ‎MPXV5100GC6U

Commit message: Add more decoupling capacitors,  clean-up some traces, add more stitching vias between ground planes
Parts:
- U6: symbol index:‎MPXV5100GC6U -> mobo-rescue:‎MPXV5100GC6U-index
Changed lines of the file:
@@
 $EndComp
 $Comp
-L index:‎MPXV5100GC6U U6
+L mobo-rescue:‎MPXV5100GC6U-index U6
 U 1 1 5F24439C
 P 3850 2000
