File: pnp/pcb/mobo/misc_output.sch (KiCad schematic (older format))
At the start: 37 parts, among them J10 MF3, J11 MF4, J12 DOWNWARDS_LIGHT, J13 UPWARDS_LIGHT, J14 5V_INJECTION, J15 RS-485_1, J16 RS-485_2, J17 RS-485_3, J21 I2C, J22 SPI, J23 AUX1, J24 AUX2, J6 SERVO1, J7 SERVO2, J8 MF1, J9 MF2, Q1 IRF540N, Q2 IRF540N, Q3 IRF540N, Q4 IRF540N, U2 SP3485EN, U3 SP3485EN, U4 SP3485EN

Commit message: Add more decoupling capacitors,  clean-up some traces, add more stitching vias between ground planes
Parts:
- C26, C27, C28: footprint Capacitor_SMD:C_0805_2012Metric_Pad1.15x1.40mm_HandSolder -> Capacitor_SMD:C_0805_2012Metric_Pad1.18x1.45mm_HandSolder
Changed lines of the file:
@@
 F 0 "C26" H 4942 3546 50  0000 L CNN
 F 1 "0.1uF" H 4942 3455 50  0000 L CNN
-F 2 "Capacitor_SMD:C_0805_2012Metric_Pad1.15x1.40mm_HandSolder" H 4850 3500 50  0001 C CNN
+F 2 "Capacitor_SMD:C_0805_2012Metric_Pad1.18x1.45mm_HandSolder" H 4850 3500 50  0001 C CNN
 F 3 "~" H 4850 3500 50  0001 C CNN
 	1    4850 3500
@@
 F 0 "C27" H 4942 4896 50  0000 L CNN
 F 1 "0.1uF" H 4942 4805 50  0000 L CNN
-F 2 "Capacitor_SMD:C_0805_2012Metric_Pad1.15x1.40mm_HandSolder" H 4850 4850 50  0001 C CNN
+F 2 "Capacitor_SMD:C_0805_2012Metric_Pad1.18x1.45mm_HandSolder" H 4850 4850 50  0001 C CNN
 F 3 "~" H 4850 4850 50  0001 C CNN
 	1    4850 4850
@@
 F 0 "C28" H 4942 6246 50  0000 L CNN
 F 1 "0.1uF" H 4942 6155 50  0000 L CNN
-F 2 "Capacitor_SMD:C_0805_2012Metric_Pad1.15x1.40mm_HandSolder" H 4850 6200 50  0001 C CNN
+F 2 "Capacitor_SMD:C_0805_2012Metric_Pad1.18x1.45mm_HandSolder" H 4850 6200 50  0001 C CNN
 F 3 "~" H 4850 6200 50  0001 C CNN
 	1    4850 6200
