File: pnp/pcb/mobo/power.sch (KiCad schematic (older format))
At the start: 26 parts, among them J45 Jack-DC, U5 AP1117-33, U7 TPS54336ADDA

Commit message: Add more decoupling capacitors,  clean-up some traces, add more stitching vias between ground planes
Parts:
- C10, C11, C12, C29, C31, C8, C9: footprint Capacitor_SMD:C_0805_2012Metric_Pad1.15x1.40mm_HandSolder -> Capacitor_SMD:C_0805_2012Metric_Pad1.18x1.45mm_HandSolder
Changed lines of the file:
@@
 F 0 "C8" H 2715 1446 50  0000 L CNN
 F 1 "0.1uF" H 2715 1355 50  0000 L CNN
-F 2 "Capacitor_SMD:C_0805_2012Metric_Pad1.15x1.40mm_HandSolder" H 2638 1250 50  0001 C CNN
+F 2 "Capacitor_SMD:C_0805_2012Metric_Pad1.18x1.45mm_HandSolder" H 2638 1250 50  0001 C CNN
 F 3 "~" H 2600 1400 50  0001 C CNN
 	1    2600 1400
@@
 F 0 "C12" V 5748 1300 50  0000 C CNN
 F 1 "0.1uF" V 5839 1300 50  0000 C CNN
-F 2 "Capacitor_SMD:C_0805_2012Metric_Pad1.15x1.40mm_HandSolder" H 6038 1150 50  0001 C CNN
+F 2 "Capacitor_SMD:C_0805_2012Metric_Pad1.18x1.45mm_HandSolder" H 6038 1150 50  0001 C CNN
 F 3 "~" H 6000 1300 50  0001 C CNN
 	1    6000 1300
@@
 F 0 "C11" H 4485 1854 50  0000 R CNN
 F 1 "0.01uF" H 4485 1945 50  0000 R CNN
-F 2 "Capacitor_SMD:C_0805_2012Metric_Pad1.15x1.40mm_HandSolder" H 4638 1750 50  0001 C CNN
+F 2 "Capacitor_SMD:C_0805_2012Metric_Pad1.18x1.45mm_HandSolder" H 4638 1750 50  0001 C CNN
 F 3 "~" H 4600 1900 50  0001 C CNN
 	1    4600 1900
@@
 F 0 "C10" H 4085 2004 50  0000 R CNN
 F 1 "120pF" H 4085 2095 50  0000 R CNN
-F 2 "Capacitor_SMD:C_0805_2012Metric_Pad1.15x1.40mm_HandSolder" H 4238 1900 50  0001 C CNN
+F 2 "Capacitor_SMD:C_0805_2012Metric_Pad1.18x1.45mm_HandSolder" H 4238 1900 50  0001 C CNN
 F 3 "~" H 4200 2050 50  0001 C CNN
 	1    4200 2050
@@
 F 0 "C9" H 3585 2004 50  0000 R CNN
 F 1 "0.01uF" H 3585 2095 50  0000 R CNN
-F 2 "Capacitor_SMD:C_0805_2012Metric_Pad1.15x1.40mm_HandSolder" H 3738 1900 50  0001 C CNN
+F 2 "Capacitor_SMD:C_0805_2012Metric_Pad1.18x1.45mm_HandSolder" H 3738 1900 50  0001 C CNN
 F 3 "~" H 3700 2050 50  0001 C CNN
 	1    3700 2050
@@
 F 0 "C31" H 7415 1696 50  0000 L CNN
 F 1 "0.1uF" H 7415 1605 50  0000 L CNN
-F 2 "Capacitor_SMD:C_0805_2012Metric_Pad1.15x1.40mm_HandSolder" H 7338 1500 50  0001 C CNN
+F 2 "Capacitor_SMD:C_0805_2012Metric_Pad1.18x1.45mm_HandSolder" H 7338 1500 50  0001 C CNN
 F 3 "~" H 7300 1650 50  0001 C CNN
 	1    7300 1650
@@
 F 0 "C29" H 4865 3696 50  0000 L CNN
 F 1 "0.1uF" H 4865 3605 50  0000 L CNN
-F 2 "Capacitor_SMD:C_0805_2012Metric_Pad1.15x1.40mm_HandSolder" H 4788 3500 50  0001 C CNN
+F 2 "Capacitor_SMD:C_0805_2012Metric_Pad1.18x1.45mm_HandSolder" H 4788 3500 50  0001 C CNN
 F 3 "~" H 4750 3650 50  0001 C CNN
 	1    4750 3650
